Commit message: [GZ] Fix wheel collision bounds

File: tinkerbot_gazebo_sim/description/component_macros.xacro (robot description, xacro)
@@ -13,5 +13,5 @@
             <collision>
                 <geometry>
-                    <sphere radius="${radius + 0.1}"/>
+                    <sphere radius="${radius + 0.001}"/>
                 </geometry>
             </collision>

Commit message: [GZ] Add camera to robot model

File: tinkerbot_gazebo_sim/description/component_macros.xacro (robot description, xacro)
@@ -1,5 +1,5 @@
 <?xml version="1.0"?>
-<robot xmlns:xacro="http://www.ros.org/wiki/xacro" >
-    <xacro:include filename="inertial_macros.xacro"/>
+<robot xmlns:xacro="http://www.ros.org/wiki/xacro">
+    <xacro:include filename="inertial_macros.xacro" />
     <!-- Macro for creating a wheel -->
     <xacro:macro name="wheel" params="robot_pos radius width mass">
@@ -7,15 +7,15 @@
             <visual>
                 <geometry>
-                    <cylinder radius="${radius}" length="${width}"/>
+                    <cylinder radius="${radius}" length="${width}" />
                 </geometry>
-                <material name="black"/>
+                <material name="black" />
             </visual>
             <collision>
                 <geometry>
-                    <sphere radius="${radius + 0.001}"/>
+                    <sphere radius="${radius + 0.001}" />
                 </geometry>
             </collision>
             <xacro:inertial_cylinder mass="${mass}" length="${width}" radius="${radius}">
-                <origin xyz="0.0 0.0 0.0" rpy="0 0 0"/>
+                <origin xyz="0.0 0.0 0.0" rpy="0 0 0" />
             </xacro:inertial_cylinder>
         </link>
@@ -25,18 +25,18 @@
         <link name="chassis">
             <visual>
-                <origin xyz="${length/2} 0 ${height/2}"/>
+                <origin xyz="${length/2} 0 ${height/2}" />
                 <geometry>
-                    <box size="${length} ${width} ${height}"/>
+                    <box size="${length} ${width} ${height}" />
                 </geometry>
-                <material name="white"/>
+                <material name="white" />
             </visual>
             <collision>
-                <origin xyz="${length/2} 0 ${height/2}"/>
+                <origin xyz="${length/2} 0 ${height/2}" />
                 <geometry>
-                    <box size="${length} ${width} ${height}"/>
+                    <box size="${length} ${width} ${height}" />
                 </geometry>
             </collision>
             <xacro:inertial_box mass="${mass}" x="${length}" y="${width}" z="${height}">
-                <origin xyz="${length/2} 0 ${height/2}" rpy="0.0 0.0 0.0"/>
+                <origin xyz="${length/2} 0 ${height/2}" rpy="0.0 0.0 0.0" />
             </xacro:inertial_box>
         </link>

File: tinkerbot_gazebo_sim/description/robot_core.xacro (robot description, xacro)
@@ -1,17 +1,21 @@
 <?xml version="1.0"?>
 <robot xmlns:xacro="http://www.ros.org/wiki/xacro">
-    <xacro:include filename="robot_properties.xacro"/>
-    <xacro:include filename="component_macros.xacro"/>
+    <xacro:include filename="robot_properties.xacro" />
+    <xacro:include filename="component_macros.xacro" />
+    <xacro:include filename="sensor_macros.xacro" />
     <material name="white">
-        <color rgba="1 1 1 1"/>
+        <color rgba="1 1 1 1" />
     </material>
     <material name="blue">
-        <color rgba="0 0 1 1"/>
+        <color rgba="0 0 1 1" />
     </material>
     <material name="black">
-        <color rgba="0 0 0 1"/>
+        <color rgba="0 0 0 1" />
     </material>
     <material name="green">
-        <color rgba="0 1 0 1"/>
+        <color rgba="0 1 0 1" />
+    </material>
+    <material name="red">
+        <color rgba="1 0 0 1" />
     </material>
     <!-- BASE LINK OBJECT -->
@@ -20,7 +24,7 @@
     <!-- CHASSIS OBJECT -->
     <joint name="chassis_joint" type="fixed">
-        <parent link="base_link"/>
-        <child link="chassis"/>
-        <origin xyz="-${chassis_length/2} 0.0 0.0"/>
+        <parent link="base_link" />
+        <child link="chassis" />
+        <origin xyz="-${chassis_length/2} 0.0 0.0" />
     </joint>
     <xacro:chassis
@@ -39,7 +43,7 @@
     />
     <joint name="front_left_wheel_joint" type="continuous">
-        <parent link="base_link"/>
-        <child link="front_left_wheel"/>
-        <axis xyz="0.0 0.0 1"/>
+        <parent link="base_link" />
+        <child link="front_left_wheel" />
+        <axis xyz="0.0 0.0 1" />
         <origin
             xyz="${wheel_base/2} ${track_width/2} ${wheel_z_offset}"
@@ -55,7 +59,7 @@
     />
     <joint name="front_right_wheel_joint" type="continuous">
-        <parent link="base_link"/>
-        <child link="front_right_wheel"/>
-        <axis xyz="0.0 0.0 -1"/>
+        <parent link="base_link" />
+        <child link="front_right_wheel" />
+        <axis xyz="0.0 0.0 -1" />
         <origin
             xyz="${wheel_base/2} -${track_width/2} ${wheel_z_offset}"
@@ -71,7 +75,7 @@
     />
     <joint name="back_left_wheel_joint" type="continuous">
-        <parent link="base_link"/>
-        <child link="back_left_wheel"/>
-        <axis xyz="0.0 0.0 1"/>
+        <parent link="base_link" />
+        <child link="back_left_wheel" />
+        <axis xyz="0.0 0.0 1" />
         <origin
             xyz="-${wheel_base/2} ${track_width/2} ${wheel_z_offset}"
@@ -87,7 +91,7 @@
     />
     <joint name="back_right_wheel_joint" type="continuous">
-        <parent link="base_link"/>
-        <child link="back_right_wheel"/>
-        <axis xyz="0.0 0.0 -1"/>
+        <parent link="base_link" />
+        <child link="back_right_wheel" />
+        <axis xyz="0.0 0.0 -1" />
         <origin
             xyz="-${wheel_base/2} -${track_width/2} ${wheel_z_offset}"
@@ -95,3 +99,12 @@
         />
     </joint>
+    <!-- Front webcam -->
+    <xacro:webcam
+        name="front_webcam"
+    />
+    <joint name="front_webcam_joint" type="fixed">
+        <parent link="chassis" />
+        <child link="front_webcam_link" />
+        <origin xyz="${webcam_x_offset} ${webcam_y_offset} ${webcam_z_offset}" rpy="0 0 0" />
+    </joint>
 </robot>

File: tinkerbot_gazebo_sim/description/robot_properties.xacro (robot description, xacro)
@@ -11,3 +11,6 @@
     <xacro:property name="wheel_base" value=".6" />
     <xacro:property name="wheel_z_offset" value="0.1" />
+    <xacro:property name="webcam_x_offset" value="${chassis_length}" />
+    <xacro:property name="webcam_y_offset" value="0.0" />
+    <xacro:property name="webcam_z_offset" value="${chassis_height}" />
 </robot>
