Commit message: [GZ] Add depth sensor to robot model

File: tinkerbot_gazebo_sim/description/robot_core.xacro (robot description, xacro)
@@ -108,3 +108,12 @@
         <origin xyz="${webcam_x_offset} ${webcam_y_offset} ${webcam_z_offset}" rpy="0 0 0" />
     </joint>
+    <!-- Front webcam -->
+    <xacro:depth_cam
+        name="front_depth_camera"
+    />
+    <joint name="front_depth_camera_joint" type="fixed">
+        <parent link="chassis" />
+        <child link="front_depth_camera_link" />
+        <origin xyz="${webcam_x_offset} ${webcam_y_offset} ${webcam_z_offset - 0.2}" rpy="0 0 0" />
+    </joint>
 </robot>

File: tinkerbot_gazebo_sim/description/sensor_macros.xacro (robot description, xacro)
@@ -40,3 +40,44 @@
         </gazebo>
     </xacro:macro>
+    <!-- Macro for creating depth cameras -->
+    <xacro:macro name="depth_cam" params="name">
+        <link name="${name}_link">
+            <visual>
+                <geometry>
+                    <box size="0.03 0.07 0.03" />
+                </geometry>
+                <material name="blue" />
+            </visual>
+        </link>
+        <link name="${name}_link_optical"></link>
+        <joint name="${name}_optical_joint" type="fixed">
+            <origin xyz="0 0 0" rpy="${-pi/2} 0 ${-pi/2}" />
+            <parent link="${name}_link" />
+            <child link="${name}_link_optical" />
+        </joint>
+        <gazebo reference="${name}_link">
+            <sensor name="${name}" type="depth">
+                <camera>
+                    <camera_info_topic>${name}/camera_info</camera_info_topic>
+                    <horizontal_fov>1.20</horizontal_fov>
+                    <image>
+                        <width>640</width>
+                        <height>480</height>
+                    </image>
+                    <clip>
+                        <near>0.1</near>
+                        <far>8</far>
+                    </clip>
+                </camera>
+                <always_on>1</always_on>
+                <update_rate>30</update_rate>
+                <visualize>true</visualize>
+                <topic>${name}/image_raw</topic>
+                <!-- Gazebo seems to output PointCloud data with the correct axis already -->
+                <!-- X forward, Y left, Z up -->
+                <!-- So we don't need to use the optical frame -->
+                <gz_frame_id>${name}_link</gz_frame_id>
+            </sensor>
+        </gazebo>
+    </xacro:macro>
 </robot>
